File: Hardware/mobile_receiver/mobile_receiver.kicad_pcb (KiCad board)
At the start: 4 copper layers, 82.5 x 142 mm, 33 parts, among them J1 Conn_02x07_Top_Bottom, SW1 SW_SPST, SW2 SW_Push, SW3 SW_Push, SW4 SW_Push, SW5 SW_Push, SW6 SW_Push, SW7 SW_Push, U2 kb2040

Commit message: Refined Trace Jumps
Parts:
- moved R5 1.14 mm to (206.5, 176.5)
Routing:
- net /SYS_SCK: track 97.9 -> 96.7 mm
- net +3.3V: track 147.4 -> 148.5 mm
- net Net-(J1-Pin_3): track 18.1 -> 19.2 mm
- net /VBAT: track 60.0 -> 59.1 mm
- net GND: vias 33 -> 47
