File: Hardware/CATS_adapter/CATS_adapter.kicad_pcb (KiCad board)
At the start: 2 copper layers, 99.5 x 34.5 mm, 11 parts, among them IC1 LAMBDA80C-24S, J1 Conn_01x04, J2 Conn_02x07_Top_Bottom, SW1 SW_Push, U1 STM32G071CBT6

Commit message: keep out zone added on cats
Routing:
- net GND: vias 34 -> 30
Changed lines of the file:
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@@
-	)
-	(via
-		(at 106.730964 102.737126)
-		(size 0.6)
-		(drill 0.3)
-		(layers "F.Cu" "B.Cu")
-		(free yes)
-		(net "GND")
 	)
 	(via
@@
 	)
 	(via
-		(at 100.910994 101.518993)
-		(size 0.6)
-		(drill 0.3)
-		(layers "F.Cu" "B.Cu")
-		(free yes)
-		(net "GND")
-	)
-	(via
 		(at 140.75 104.1)
 		(size 0.6)
@@
 	)
 	(via
-		(at 106.900149 95.15763)
-		(size 0.6)
-		(drill 0.3)
-		(layers "F.Cu" "B.Cu")
-		(free yes)
-		(net "GND")
-	)
-	(via
 		(at 156.531065 98.202266)
 		(size 0.6)
@@
 	(via
 		(at 172.823598 93.989555)
-		(size 0.6)
-		(drill 0.3)
-		(layers "F.Cu" "B.Cu")
-		(free yes)
-		(net "GND")
-	)
-	(via
-		(at 101.75692 94.5824)
 		(size 0.6)
 		(drill 0.3)
@@
 	)
 	(zone
+		(layer "F.Cu")
+		(hatch edge 0.5)
+		(connect_pads
+			(clearance 0)
+		)
+		(min_thickness 0.25)
+		(keepout
+			(tracks not_allowed)
+			(vias not_allowed)
+			(pads not_allowed)
+			(copperpour not_allowed)
+			(footprints allowed)
+		)
+		(placement
+			(enabled no)
+			(sheetname "/")
+		)
+		(fill
+			(thermal_gap 0.5)
+			(thermal_bridge_width 0.5)
+			(island_removal_mode 0)
+		)
+		(polygon
+			(pts
+				(xy 98.65 78.75) (xy 109.425168 78.69417) (xy 109.574968 118.141352) (xy 97.9 118.75)
+			)
+		)
+	)
+	(zone

Commit message: CATS changes made: bac keepout zone, 3.3V vref etc..
Parts:
- J1: value Conn_01x04 -> Conn_01x05; footprint Connector_PinHeader_2.54mm:PinHeader_1x04_P2.54mm_Vertical -> Connector_PinHeader_2.54mm:PinHeader_1x05_P2.54mm_Vertical
- U1: footprint My Feetpics:LQFP-48-L -> Package_QFP:LQFP-48_7x7mm_P0.5mm
- moved J1 2.56 mm to (165.1, 110.6)
Connections:
- J1 pad 2: /SWCLK -> +3.3V
- J1 pad 3: /SWDIO -> /SWCLK
- J1 pad 4: /NRST -> /SWDIO
Routing:
- net +3.3V: track 122.3 -> 134.1 mm
- net GND: track 0.00 -> 1.81 mm

Commit message: added logo to cats
Parts:
- added G***: LOGO, MHF4_antenna:HiPR, F.Cu at (119.0, 85.0)
Routing:
- net GND: vias 30 -> 34
